Commit message: Add files via upload

File: single_swerve_robot/description/swerve_bot.urdf (robot description, URDF)
Before this commit: robot swerve_bot, 4 links, 3 joints
Links:
- link lidar_link: geometry visual box size=0.05 0.05 0.05
Joints:
- joint lidar_joint: origin xyz=0.2555 0 0.1156 rpy=0 0 0 -> xyz=0.2555 0 0.05 rpy=0.0 0.0 0.0
